Commit message: edit gazebo camera plugin and enable to reach visual odom

File: src/rover_description/urdf/_d435.gazebo.xacro (robot description, xacro)
@@ -6,8 +6,8 @@
 -->
 <robot xmlns:xacro="http://ros.org/wiki/xacro">
-  <xacro:macro name="gazebo_d435" params="camera_name reference_link topics_ns depth_optical_frame color_optical_frame infrared1_optical_frame infrared2_optical_frame publish_pointcloud:=true" >
+  <xacro:macro name="gazebo_d435" params="camera_name  topics_ns depth_optical_frame color_optical_frame infrared1_optical_frame infrared2_optical_frame publish_pointcloud:=true" >
     <!-- Load parameters to model's main link-->
     <xacro:property name="deg_to_rad" value="0.01745329251994329577" />
-    <gazebo reference="${reference_link}">
+    <gazebo reference="camera_attachment_link">
       <self_collide>0</self_collide>
       <enable_wind>0</enable_wind>
@@ -23,5 +23,5 @@
       <!--<max_vel>0.01</max_vel>
       <min_depth>0</min_depth>-->
-      <sensor name="${camera_name}color" type="camera">
+      <sensor name="${camera_name}_color" type="camera">
         <camera name="${camera_name}">
           <horizontal_fov>${69.4*deg_to_rad}</horizontal_fov>
@@ -44,6 +44,17 @@
         <update_rate>30</update_rate>
         <visualize>1</visualize>
+        <plugin name="${camera_name}_color" filename="libgazebo_ros_camera.so">
+          <alwaysOn>true</alwaysOn>
+          <updateRate>0.0</updateRate>
+          <frame_name>${name}_color_optical_frame</frame_name>
+          <hackBaseline>0.07</hackBaseline>
+          <distortionK1>0.0</distortionK1>
+          <distortionK2>0.0</distortionK2>
+          <distortionK3>0.0</distortionK3>
+          <distortionT1>0.0</distortionT1>
+          <distortionT2>0.0</distortionT2>
+        </plugin>
       </sensor>
-      <sensor name="${camera_name}ired1" type="camera">
+      <sensor name="${camera_name}_ired1" type="camera">
         <camera name="${camera_name}">
           <horizontal_fov>${85.2*deg_to_rad}</horizontal_fov>
@@ -66,6 +77,22 @@
         <update_rate>90</update_rate>
         <visualize>0</visualize>
+        <plugin name="${camera_name}_ired1" filename="libgazebo_ros_camera.so">
+          <alwaysOn>true</alwaysOn>
+          <updateRate>0.0</updateRate>
+          <ros>
+            <remapping>/stereo_camera_ired1/image_raw:=/stereo_camera/infra1/image_rect</remapping>
+            <remapping>/stereo_camera_ired1/camera_info:=/stereo_camera/infra1/camera_info</remapping>
+          </ros>
+          <cameraInfoTopicName>/infra1/camera_info</cameraInfoTopicName>
+          <frame_name>${name}_left_ir_optical_frame</frame_name>
+          <hackBaseline>0.07</hackBaseline>
+          <distortionK1>0.0</distortionK1>
+          <distortionK2>0.0</distortionK2>
+          <distortionK3>0.0</distortionK3>
+          <distortionT1>0.0</distortionT1>
+          <distortionT2>0.0</distortionT2>
+        </plugin>
       </sensor>
-      <sensor name="${camera_name}ired2" type="camera">
+      <sensor name="${camera_name}_ired2" type="camera">
         <camera name="${camera_name}">
           <horizontal_fov>${85.2*deg_to_rad}</horizontal_fov>
@@ -88,4 +115,20 @@
         <update_rate>90</update_rate>
         <visualize>0</visualize>
+        <plugin name="${camera_name}_ired2" filename="libgazebo_ros_camera.so">
+          <alwaysOn>true</alwaysOn>
+          <updateRate>0.0</updateRate>
+          <cameraName>${camera_name}_ired2</cameraName>
+          <ros>
+            <remapping>/stereo_camera_ired2/image_raw:=/stereo_camera/infra2/image_rect</remapping>
+            <remapping>/stereo_camera_ired2/camera_info:=/stereo_camera/infra2/camera_info</remapping>
+          </ros>
+          <frame_name>${name}_right_ir_optical_frame</frame_name>
+          <hackBaseline>0.07</hackBaseline>
+          <distortionK1>0.0</distortionK1>
+          <distortionK2>0.0</distortionK2>
+          <distortionK3>0.0</distortionK3>
+          <distortionT1>0.0</distortionT1>
+          <distortionT2>0.0</distortionT2>
+        </plugin>
       </sensor>
       <sensor name="${camera_name}depth" type="depth">
@@ -95,4 +138,5 @@
             <width>1280</width>
             <height>720</height>
+            <format>R8G8B8</format>
           </image>
           <clip>
@@ -109,31 +153,19 @@
         <update_rate>90</update_rate>
         <visualize>0</visualize>
+        <plugin name="${camera_name}depth" filename="libgazebo_ros_camera.so">
+          <alwaysOn>true</alwaysOn>
+          <updateRate>0.0</updateRate>
+          <cameraName>${camera_name}depth</cameraName>
+          <imageTopicName>/depth/image_raw</imageTopicName>
+          <cameraInfoTopicName>/depth/camera_info</cameraInfoTopicName>
+          <frame_name>${name}_depth_optical_frame</frame_name>
+          <hackBaseline>0.07</hackBaseline>
+          <distortionK1>0.0</distortionK1>
+          <distortionK2>0.0</distortionK2>
+          <distortionK3>0.0</distortionK3>
+          <distortionT1>0.0</distortionT1>
+          <distortionT2>0.0</distortionT2>
+        </plugin>
       </sensor>
-    </gazebo>
-    <gazebo>
-      <plugin name="${topics_ns}" filename="librealsense_gazebo_plugin.so">
-        <prefix>${camera_name}</prefix>
-        <depthUpdateRate>30.0</depthUpdateRate>
-        <colorUpdateRate>30.0</colorUpdateRate>
-        <infraredUpdateRate>30.0</infraredUpdateRate>
-        <depthTopicName>depth/image_raw</depthTopicName>
-        <depthCameraInfoTopicName>depth/camera_info</depthCameraInfoTopicName>
-        <colorTopicName>color/image_raw</colorTopicName>
-        <colorCameraInfoTopicName>color/camera_info</colorCameraInfoTopicName>
-        <infrared1TopicName>infra1/image_raw</infrared1TopicName>
-        <infrared1CameraInfoTopicName>infra1/camera_info</infrared1CameraInfoTopicName>
-        <infrared2TopicName>infra2/image_raw</infrared2TopicName>
-        <infrared2CameraInfoTopicName>infra2/camera_info</infrared2CameraInfoTopicName>
-        <colorOpticalframeName>${color_optical_frame}</colorOpticalframeName>
-        <depthOpticalframeName>${depth_optical_frame}</depthOpticalframeName>
-        <infrared1OpticalframeName>${infrared1_optical_frame}</infrared1OpticalframeName>
-        <infrared2OpticalframeName>${infrared2_optical_frame}</infrared2OpticalframeName>
-        <rangeMinDepth>0.2</rangeMinDepth>
-        <rangeMaxDepth>10.0</rangeMaxDepth>
-        <pointCloud>${publish_pointcloud}</pointCloud>
-        <pointCloudTopicName>depth/color/points</pointCloudTopicName>
-        <pointCloudCutoff>0.25</pointCloudCutoff>
-        <pointCloudCutoffMax>9.0</pointCloudCutoffMax>
-      </plugin>
     </gazebo>
   </xacro:macro>

File: src/rover_description/urdf/_d435.urdf.xacro (robot description, xacro)
@@ -6,5 +6,5 @@
 aluminum peripherial evaluation case.
 -->
-<robot name="camera" xmlns:xacro="http://ros.org/wiki/xacro">
+<robot name="stereo_camera" xmlns:xacro="http://ros.org/wiki/xacro">
   <!--File includes-->
   <xacro:include filename="$(find rover_description)/urdf/_d435.gazebo.xacro"/>
@@ -49,5 +49,5 @@
           <!-- <box size="${d435_cam_width} ${d435_cam_height} ${d435_cam_depth}"/> -->
           <!-- <mesh filename="package://realsense2_description/meshes/d435.dae" /> -->
-          <mesh filename="file://$(find realsense2_description)/meshes/d435.dae" scale="1 1 1"/>
+          <mesh filename="file://$(find rover_description)/meshes/d435.dae" scale="1 1 1"/>
         </geometry>
         <material name="${name}_aluminum"/>
@@ -119,5 +119,5 @@
     <link name="${name}_color_optical_frame"/>
     <!-- Realsense Gazebo Plugin -->
-    <xacro:gazebo_d435 camera_name="${name}" reference_link="${name}_link" topics_ns="${topics_ns}" depth_optical_frame="${name}_depth_optical_frame" color_optical_frame="${name}_color_optical_frame" infrared1_optical_frame="${name}_left_ir_optical_frame" infrared2_optical_frame="${name}_right_ir_optical_frame" publish_pointcloud="${publish_pointcloud}"/>
+    <xacro:gazebo_d435 camera_name="${name}" topics_ns="stereo_camera" depth_optical_frame="${name}_depth_optical_frame" color_optical_frame="${name}_color_optical_frame" infrared1_optical_frame="${name}_left_ir_optical_frame" infrared2_optical_frame="${name}_right_ir_optical_frame" publish_pointcloud="${publish_pointcloud}"/>
   </xacro:macro>
 </robot>

File: src/rover_description/urdf/rover_description.xacro (robot description, xacro)
@@ -1,5 +1,5 @@
 <?xml version="1.0" ?>
 <robot name="rover" xmlns:xacro="http://www.ros.org/wiki/xacro">
-<xacro:include filename="$(find realsense2_description)/urdf/_d435.urdf.xacro" />
+<!-- <xacro:include filename="$(find realsense2_description)/urdf/_d435.urdf.xacro" /> -->
 <link name="base_link">
   <inertial>
@@ -178,3 +178,10 @@
   <axis xyz="0.0 -1.0 0.0"/>
 </joint>
+  <link name="camera_attachment_link"></link>
+    <joint name="camera_attachment_joint" type="fixed">
+      <axis xyz="0 1 0" />
+      <origin xyz="0.36 0.0 0.35" rpy="0 0 0"/>
+      <parent link="base_link"/>
+      <child link="camera_attachment_link"/>
+    </joint>
 </robot>

File: src/rover_description/urdf/rover_realsense.xacro (robot description, xacro)
@@ -30,5 +30,5 @@
     <child link="camera_link"/>
     </joint>
-    <xacro:sensor_d435 name="depthcamera" parent="camera_link">
+    <xacro:sensor_d435 name="stereo_camera" parent="camera_link">
     <origin xyz="0.0 0.0 0.05" rpy="0 0 0" />
     </xacro:sensor_d435>
