Commit message: clean urdf folder

File: src/rover_description/urdf/rover.xacro (robot description, xacro)
@@ -1,5 +1,4 @@
 <?xml version="1.0" ?>
 <robot name="rover" xmlns:xacro="http://www.ros.org/wiki/xacro">
-  <xacro:include filename="$(find rover_description)/urdf/materials.xacro" />
   <xacro:include filename="$(find rover_description)/urdf/rover.trans" />
   <xacro:include filename="$(find rover_description)/urdf/rover_description.xacro" />

File: src/rover_description/urdf/rover_camera.xacro (robot description, xacro)
@@ -1,35 +1,46 @@
 <?xml version="1.0" ?>
 <robot name="rover" xmlns:xacro="http://www.ros.org/wiki/xacro">
-    <xacro:include filename="$(find rover_description)/urdf/stereo.urdf.xacro" />
+    <xacro:include filename="$(find rover_description)/urdf/stereo.gazebo.xacro"/>
+    <xacro:property name="M_PI" value="3.1415926535897931" />
     <link name="camera_link">
-    <collision>
+      <collision>
         <origin xyz="0 0 0" rpy="0 0 0"/>
         <geometry>
-    <box size="0.01 0.01 0.01"/>
+          <box size="0.01 0.01 0.01"/>
         </geometry>
-    </collision>
-    <visual>
+      </collision>
+      <visual>
         <origin xyz="0 0 0" rpy="0 0 0"/>
         <geometry>
-    <box size="0.01 0.01 0.01"/>
+          <box size="0.01 0.01 0.01"/>
         </geometry>
         <material name="silver">
-        <color rgba="0.700 0.700 0.700 1.000"/>
+          <color rgba="0.700 0.700 0.700 1.000"/>
         </material>
-    </visual>
-    <inertial>
+      </visual>
+      <inertial>
         <mass value="1e-5" />
         <origin xyz="0 0 0" rpy="0 0 0"/>
         <inertia ixx="1e-6" ixy="0" ixz="0" iyy="1e-6" iyz="0" izz="1e-6" />
-    </inertial>
+      </inertial>
     </link>
     <joint name="camera_joint" type="fixed">
-    <axis xyz="0 1 0" />
-    <origin xyz="0.33 0.0 0.35" rpy="0 0 0"/>
-    <parent link="base_link"/>
-    <child link="camera_link"/>
+      <axis xyz="0 1 0" />
+      <origin xyz="0.33 0.0 0.4" rpy="0 0 0"/>
+      <parent link="base_link"/>
+      <child link="camera_link"/>
     </joint>
-    <xacro:sensor_d435 name="stereo_camera" parent="camera_link">
-    <origin xyz="0.0 0.0 0.05" rpy="0 0 0" />
-    </xacro:sensor_d435>
+    <joint name="left_optical_joint" type="fixed">
+      <origin xyz="0 0 0" rpy="${-M_PI/2} 0 ${-M_PI/2}" />
+      <parent link="camera_link" />
+      <child link="stereo_camera_left_frame" />
+    </joint>
+    <link name="stereo_camera_left_frame"/>
+    <joint name="stereo_camera_right_joint" type="fixed">
+      <origin xyz="0 -0.05 0" rpy="${-M_PI/2} 0 ${-M_PI/2}" />
+      <parent link="camera_link" />
+      <child link="stereo_camera_right_frame" />
+    </joint>
+    <link name="stereo_camera_right_frame"/>
+    <xacro:gazebo_d435 topics_ns="stereo_camera" />
 </robot>

File: src/rover_description/urdf/rover_description.xacro (robot description, xacro)
@@ -2,4 +2,7 @@
 <robot name="rover" xmlns:xacro="http://www.ros.org/wiki/xacro">
 <!-- <xacro:include filename="$(find realsense2_description)/urdf/_d435.urdf.xacro" /> -->
+<material name="silver">
+  <color rgba="0.700 0.700 0.700 1.000"/>
+</material>
 <link name="base_link">
   <inertial>

File: src/rover_description/urdf/stereo.gazebo.xacro (robot description, xacro)
@@ -6,10 +6,10 @@
 -->
 <robot xmlns:xacro="http://ros.org/wiki/xacro">
-  <xacro:macro name="gazebo_d435" params="camera_name  topics_ns depth_optical_frame color_optical_frame infrared1_optical_frame infrared2_optical_frame publish_pointcloud:=true" >
+  <xacro:macro name="gazebo_d435" params="topics_ns" >
     <!-- Load parameters to model's main link-->
     <xacro:property name="deg_to_rad" value="0.01745329251994329577" />
-    <gazebo reference="${name}_left_ir_frame">
-      <sensor name="${camera_name}_ired1" type="camera">
-        <camera name="${camera_name}">
+    <gazebo reference="stereo_camera_left_frame">
+      <sensor name="stereo_camera_left" type="camera">
+        <camera name="stereo_camera_left">
           <horizontal_fov>${85.2*deg_to_rad}</horizontal_fov>
           <image>
@@ -31,13 +31,12 @@
         <update_rate>90</update_rate>
         <visualize>0</visualize>
-        <plugin name="${camera_name}_ired1" filename="libgazebo_ros_camera.so">
+        <plugin name="stereo_camera_left" filename="libgazebo_ros_camera.so">
           <alwaysOn>true</alwaysOn>
           <updateRate>0.0</updateRate>
           <ros>
-            <remapping>/stereo_camera_ired1/image_raw:=/stereo_camera/infra1/image_raw</remapping>
-            <remapping>/stereo_camera_ired1/camera_info:=/stereo_camera/infra1/camera_info</remapping>
+            <remapping>/stereo_camera_left/image_raw:=/stereo_camera/left/image_raw</remapping>
+            <remapping>/stereo_camera_left/camera_info:=/stereo_camera/left/camera_info</remapping>
           </ros>
-          <cameraInfoTopicName>/infra1/camera_info</cameraInfoTopicName>
-          <frame_name>${name}_left_ir_optical_frame</frame_name>
+          <frame_name>stereo_camera_left_frame</frame_name>
           <hackBaseline>0.07</hackBaseline>
           <distortionK1>0.0</distortionK1>
@@ -49,7 +48,7 @@
       </sensor>
     </gazebo>
-    <gazebo reference="${name}_right_ir_frame">
-      <sensor name="${camera_name}_ired2" type="camera">
-        <camera name="${camera_name}">
+    <gazebo reference="stereo_camera_right_frame">
+      <sensor name="stereo_camera_right" type="camera">
+        <camera name="stereo_camera_right">
           <horizontal_fov>${85.2*deg_to_rad}</horizontal_fov>
           <image>
@@ -71,13 +70,13 @@
         <update_rate>90</update_rate>
         <visualize>0</visualize>
-        <plugin name="${camera_name}_ired2" filename="libgazebo_ros_camera.so">
+        <plugin name="stereo_camera_right" filename="libgazebo_ros_camera.so">
           <alwaysOn>true</alwaysOn>
           <updateRate>0.0</updateRate>
-          <cameraName>${camera_name}_ired2</cameraName>
+          <cameraName>stereo_camera_right</cameraName>
           <ros>
-            <remapping>/stereo_camera_ired2/image_raw:=/stereo_camera/infra2/image_raw</remapping>
-            <remapping>/stereo_camera_ired2/camera_info:=/stereo_camera/infra2/camera_info</remapping>
+            <remapping>/stereo_camera_right/image_raw:=/stereo_camera/right/image_raw</remapping>
+            <remapping>/stereo_camera_right/camera_info:=/stereo_camera/right/camera_info</remapping>
           </ros>
-          <frame_name>${name}_right_ir_optical_frame</frame_name>
+          <frame_name>stereo_camera_right_frame</frame_name>
           <hackBaseline>0.07</hackBaseline>
           <distortionK1>0.0</distortionK1>

File: src/rover_description/urdf/stereo.urdf.xacro (robot description, xacro)
@@ -80,5 +80,5 @@
     <link name="${name}_depth_optical_frame"/>
     <!-- camera left IR joints and links -->
-    <joint name="${name}_left_ir_joint" type="fixed">
+    <!-- <joint name="${name}_left_ir_joint" type="fixed">
       <origin xyz="0 ${d435_cam_depth_to_left_ir_offset} 0" rpy="0 0 0" />
       <parent link="${name}_depth_frame" />
@@ -91,7 +91,7 @@
       <child link="${name}_left_ir_optical_frame" />
     </joint>
-    <link name="${name}_left_ir_optical_frame"/>
+    <link name="${name}_left_ir_optical_frame"/> -->
     <!-- camera right IR joints and links -->
-    <joint name="${name}_right_ir_joint" type="fixed">
+    <!-- <joint name="${name}_right_ir_joint" type="fixed">
       <origin xyz="0 ${d435_cam_depth_to_right_ir_offset} 0" rpy="0 0 0" />
       <parent link="${name}_depth_frame" />
@@ -104,5 +104,5 @@
       <child link="${name}_right_ir_optical_frame" />
     </joint>
-    <link name="${name}_right_ir_optical_frame"/>
+    <link name="${name}_right_ir_optical_frame"/> -->
     <!-- camera color joints and links -->
     <joint name="${name}_color_joint" type="fixed">
@@ -118,4 +118,16 @@
     </joint>
     <link name="${name}_color_optical_frame"/>
+    <joint name="${name}_left_ir_optical_joint" type="fixed">
+      <origin xyz="0 0 0" rpy="${-M_PI/2} 0 ${-M_PI/2}" />
+      <parent link="${parent}" />
+      <child link="${name}_left_ir_optical_frame" />
+    </joint>
+    <link name="${name}_left_ir_optical_frame"/>
+    <joint name="${name}_right_ir_optical_joint" type="fixed">
+      <origin xyz="0 -0.05 0" rpy="${-M_PI/2} 0 ${-M_PI/2}" />
+      <parent link="${parent}" />
+      <child link="${name}_right_ir_optical_frame" />
+    </joint>
+    <link name="${name}_right_ir_optical_frame"/>
     <!-- Realsense Gazebo Plugin -->
     <xacro:gazebo_d435 camera_name="${name}" topics_ns="stereo_camera" depth_optical_frame="${name}_depth_optical_frame" color_optical_frame="${name}_color_optical_frame" infrared1_optical_frame="${name}_left_ir_optical_frame" infrared2_optical_frame="${name}_right_ir_optical_frame" publish_pointcloud="${publish_pointcloud}"/>
