Commit message: modified update rate params

File: src/rover_description/urdf/rgbd.gazebo.xacro (robot description, xacro)
@@ -1,2 +1,3 @@
+<?xml version="1.0"?>
 <robot xmlns:xacro="http://ros.org/wiki/xacro">
     <!-- Load parameters to model's main link-->
@@ -16,5 +17,5 @@
     </joint>
     <joint name="camera_to_depth" type="fixed">
-      <origin xyz="0.01 0.0 0.0" rpy="-1.5707 0 -1.5707"/>
+      <origin xyz="0.02 0.0 0.0" rpy="-1.5707 0 -1.5707"/>
       <parent link="camera_link"/>
       <child link="depth_link"/>
@@ -42,9 +43,9 @@
         </camera>
         <always_on>1</always_on>
-        <update_rate>90</update_rate>
+        <update_rate>30</update_rate>
         <visualize>0</visualize>
         <plugin name="color" filename="libgazebo_ros_camera.so">
           <alwaysOn>true</alwaysOn>
-          <updateRate>0.0</updateRate>
+          <updateRate>30.0</updateRate>
           <frame_name>depth_link</frame_name>
           <hackBaseline>0.07</hackBaseline>
@@ -58,8 +59,13 @@
     </gazebo>
     <gazebo reference="camera_link">
-        <sensor type="depth" name="sensor_name">
+        <sensor type="depth" name="depth">
           <always_on>0</always_on>
-          <update_rate>1</update_rate>
+          <update_rate>30</update_rate>
           <camera name="depth">
+            <image>
+              <width>1280</width>
+              <height>720</height>
+              <format>R8G8B8</format>
+            </image>
             <horizontal_fov>1.57</horizontal_fov>
             <distortion>

Commit message: resolve conflicts

File: src/rover_description/urdf/rgbd.gazebo.xacro (robot description, xacro)
@@ -2,20 +2,13 @@
 <robot xmlns:xacro="http://ros.org/wiki/xacro">
     <!-- Load parameters to model's main link-->
-    <link name="camera_link">
-      <visual>
-        <origin xyz="0 0 0" rpy="-1.57 0 -1.57"/>
-        <geometry>
-          <mesh filename="file://$(find realsense2_description)/meshes/d435.dae" />
-        </geometry>
-      </visual>
-    </link>
+    <link name="camera_link"/>
     <link name="depth_link"/>
     <joint name="base_to_camera" type="fixed">
-      <origin xyz="0.34 0.0 0.4" rpy="0 0 0"/>
+      <origin xyz="0.35 0.0 0.4" rpy="0 0 0"/>
       <parent link="base_link"/>
       <child link="camera_link"/>
     </joint>
     <joint name="camera_to_depth" type="fixed">
-      <origin xyz="0.02 0.0 0.0" rpy="-1.5707 0 -1.5707"/>
+      <origin xyz="0.0 0.0 0.0" rpy="-1.5707 0 -1.5707"/>
       <parent link="camera_link"/>
       <child link="depth_link"/>
@@ -43,5 +36,5 @@
         </camera>
         <always_on>1</always_on>
-        <update_rate>30</update_rate>
+        <update_rate>10</update_rate>
         <visualize>0</visualize>
         <plugin name="color" filename="libgazebo_ros_camera.so">
@@ -58,8 +51,9 @@
       </sensor>
     </gazebo>
+    <!-- mimic realsense d435 ability -->
     <gazebo reference="camera_link">
         <sensor type="depth" name="depth">
           <always_on>0</always_on>
-          <update_rate>30</update_rate>
+          <update_rate>10</update_rate>
           <camera name="depth">
             <image>
@@ -81,6 +75,6 @@
             <frame_name>depth_link</frame_name>
             <hack_baseline>0.07</hack_baseline>
-            <min_depth>0.001</min_depth>
-            <max_depth>300.0</max_depth>
+            <min_depth>0.4</min_depth>
+            <max_depth>20.0</max_depth>
           </plugin>
         </sensor>

File: src/rover_description/urdf/rover.xacro (robot description, xacro)
@@ -5,3 +5,4 @@
   <xacro:include filename="$(find rover_description)/urdf/diff_control.xacro" />
   <xacro:include filename="$(find rover_description)/urdf/rgbd.gazebo.xacro" />
+  <xacro:include filename="$(find rover_description)/urdf/imu.gazebo.xacro" />
 </robot>
