Commit message: activate imu plugin

File: src/rover_description/urdf/imu.gazebo.xacro (robot description, xacro)
@@ -1,5 +1,32 @@
 <?xml version="1.0"?>
 <robot xmlns:xacro="http://ros.org/wiki/xacro">
-    <xacro:macro name="gazebo_d435" params="topics_ns" >
+    <link name="imu_link">
+      <collision>
+        <origin xyz="0 0 0" rpy="0 0 0"/>
+        <geometry>
+          <box size="0.01 0.01 0.01"/>
+        </geometry>
+      </collision>
+      <visual>
+        <origin xyz="0 0 0" rpy="0 0 0"/>
+        <geometry>
+          <box size="0.01 0.01 0.01"/>
+        </geometry>
+        <material name="silver">
+          <color rgba="0.700 0.700 0.700 1.000"/>
+        </material>
+      </visual>
+      <inertial>
+        <mass value="1e-5" />
+        <origin xyz="0 0 0" rpy="0 0 0"/>
+        <inertia ixx="1e-6" ixy="0" ixz="0" iyy="1e-6" iyz="0" izz="1e-6" />
+      </inertial>
+    </link>
+    <joint name="imu_joint" type="fixed">
+      <axis xyz="0 1 0" />
+      <origin xyz="0. 0.0 0.5" rpy="0 0 0"/>
+      <parent link="base_link"/>
+      <child link="imu_link"/>
+    </joint>
     <gazebo reference="imu_link">
         <gravity>true</gravity>
@@ -10,5 +37,7 @@
         <topic>__default_topic__</topic>
         <plugin filename="libgazebo_ros_imu_sensor.so" name="imu_plugin">
-            <topicName>imu</topicName>
+            <ros>
+                <remapping>/imu_plugin/out:=/imu</remapping>
+            </ros>
             <bodyName>imu_link</bodyName>
             <updateRateHZ>10.0</updateRateHZ>
@@ -22,4 +51,3 @@
         </sensor>
     </gazebo>
-    </xacro:macro>
 </robot>
