Commit message: attach realsense

File: src/rover_description/urdf/diff_control.xacro (robot description, xacro)
@@ -1,28 +1,34 @@
 <?xml version="1.0"?>
 <robot name="rover" xmlns:xacro="http://www.ros.org/wiki/xacro">
-    <gazebo>
-      <plugin filename="libgazebo_ros2_control.so" name="gazebo_ros2_control">
-        <robot_sim_type>gazebo_ros2_control/GazeboSystem</robot_sim_type>
-        <parameters>$(find rover_description)/config/diff_robot.yaml</parameters>
-      </plugin>
-    </gazebo>
-    <ros2_control name="rover" type="system">
-      <hardware>
-        <plugin>gazebo_ros2_control/GazeboSystem</plugin>
-      </hardware>
-      <hardware>
-        <plugin>mock_components/GenericSystem</plugin>
-        <param name="calculate_dynamics">true</param>
-      </hardware>
-      <joint name="left_front">
-        <command_interface name="velocity"/>
-        <state_interface name="position"/>
-        <state_interface name="velocity"/>
-      </joint>
-      <joint name="right_front">
-        <command_interface name="velocity"/>
-        <state_interface name="position"/>
-        <state_interface name="velocity"/>
-      </joint>
-    </ros2_control>
+  <gazebo>
+    <plugin filename="libgazebo_ros2_control.so" name="gazebo_ros2_control">
+      <robot_sim_type>gazebo_ros2_control/GazeboSystem</robot_sim_type>
+      <parameters>$(find rover_description)/config/diff_robot.yaml</parameters>
+      <ros>
+        <remapping>/diff_drive_controller/cmd_vel_unstamped:=/cmd_vel</remapping>
+        <remapping>/diff_drive_controller/odom:=/odom</remapping>
+      </ros>
+    </plugin>
+  </gazebo>
+  <ros2_control name="GazeboSystem" type="system">
+    <hardware>
+      <plugin>gazebo_ros2_control/GazeboSystem</plugin>
+    </hardware>
+    <joint name="left_front">
+      <command_interface name="velocity">
+        <param name="min">-1</param>
+        <param name="max">1</param>
+      </command_interface>
+      <state_interface name="position"/>
+      <state_interface name="velocity"/>
+    </joint>
+    <joint name="right_front">
+      <command_interface name="velocity">
+        <param name="min">-1</param>
+        <param name="max">1</param>
+      </command_interface>
+      <state_interface name="position"/>
+      <state_interface name="velocity"/>
+    </joint>
+  </ros2_control>
 </robot>

File: src/rover_description/urdf/rover.xacro (robot description, xacro)
@@ -5,3 +5,5 @@
   <xacro:include filename="$(find rover_description)/urdf/rover.gazebo" />
   <xacro:include filename="$(find rover_description)/urdf/rover_description.xacro" />
+  <xacro:include filename="$(find rover_description)/urdf/diff_control.xacro" />
+  <xacro:include filename="$(find rover_description)/urdf/rover_realsense.xacro" />
 </robot>

File: src/rover_description/urdf/rover_description.xacro (robot description, xacro)
@@ -166,5 +166,5 @@
   <axis xyz="0.0 1.0 -0.0"/>
 </joint>
-<joint name="link_left" type="continuous">
+<joint name="link_left" type="fixed">
   <origin xyz="0.0 0.19 0.405" rpy="0 0 0"/>
   <parent link="base_link"/>
@@ -172,5 +172,5 @@
   <axis xyz="0.0 1.0 -0.0"/>
 </joint>
-<joint name="link_right" type="continuous">
+<joint name="link_right" type="fixed">
   <origin xyz="0.0 -0.19 0.405" rpy="0 0 0"/>
   <parent link="base_link"/>
@@ -178,73 +178,3 @@
   <axis xyz="0.0 -1.0 0.0"/>
 </joint>
-  <!-- Camera -->
-  <xacro:property name="camera_link" value="0.05" /> <!-- Size of square 'camera' box -->
-  <joint name="camera_joint" type="fixed">
-    <axis xyz="0 1 0" />
-    <origin xyz="0.33 0.0 0.35" rpy="0 0 0"/>
-    <parent link="base_link"/>
-    <child link="camera_link"/>
-  </joint>
-  <link name="camera_link">
-    <collision>
-      <origin xyz="0 0 0" rpy="0 0 0"/>
-      <geometry>
-    <box size="${camera_link} ${camera_link} ${camera_link}"/>
-      </geometry>
-    </collision>
-    <visual>
-      <origin xyz="0 0 0" rpy="0 0 0"/>
-      <geometry>
-    <box size="${camera_link} ${camera_link} ${camera_link}"/>
-      </geometry>
-      <material name="red"/>
-    </visual>
-    <inertial>
-      <mass value="1e-5" />
-      <origin xyz="0 0 0" rpy="0 0 0"/>
-      <inertia ixx="1e-6" ixy="0" ixz="0" iyy="1e-6" iyz="0" izz="1e-6" />
-    </inertial>
-  </link>
-   <gazebo reference="camera_link">
-    <sensor type="camera" name="camera1">
-      <update_rate>30.0</update_rate>
-      <camera name="head">
-        <horizontal_fov>1.3962634</horizontal_fov>
-        <image>
-          <width>640</width>
-          <height>320</height>
-          <format>R8G8B8</format>
-        </image>
-        <clip>
-          <near>0.02</near>
-          <far>300</far>
-        </clip>
-        <noise>
-          <type>gaussian</type>
-          <!-- Noise is sampled independently per pixel on each frame.
-               That pixel's noise value is added to each of its color
-               channels, which at that point lie in the range [0,1]. -->
-          <mean>0.0</mean>
-          <stddev>0.007</stddev>
-        </noise>
-      </camera>
-      <plugin name="camera_controller" filename="libgazebo_ros_camera.so">
-        <alwaysOn>true</alwaysOn>
-        <updateRate>0.0</updateRate>
-        <cameraName>camera1</cameraName>
-        <imageTopicName>image_raw</imageTopicName>
-        <cameraInfoTopicName>camera_info</cameraInfoTopicName>
-        <frameName>camera_link</frameName>
-        <hackBaseline>0.07</hackBaseline>
-        <distortionK1>0.0</distortionK1>
-        <distortionK2>0.0</distortionK2>
-        <distortionK3>0.0</distortionK3>
-        <distortionT1>0.0</distortionT1>
-        <distortionT2>0.0</distortionT2>
-      </plugin>
-    </sensor>
-  </gazebo>
-<xacro:sensor_d435 name="depthcamera" parent="camera_link">
-  <origin xyz="0.0 0.0 0.0" rpy="0 0 0" />
-</xacro:sensor_d435>
 </robot>

Commit message: add rgbd.gazebo.xacro & implemeted skid steer

File: src/rover_description/urdf/diff_control.xacro (robot description, xacro)
@@ -31,4 +31,20 @@
       <state_interface name="velocity"/>
     </joint>
+    <joint name="left_back">
+      <command_interface name="velocity">
+        <param name="min">-1</param>
+        <param name="max">1</param>
+      </command_interface>
+      <state_interface name="position"/>
+      <state_interface name="velocity"/>
+    </joint>
+    <joint name="right_back">
+      <command_interface name="velocity">
+        <param name="min">-1</param>
+        <param name="max">1</param>
+      </command_interface>
+      <state_interface name="position"/>
+      <state_interface name="velocity"/>
+    </joint>
   </ros2_control>
 </robot>

File: src/rover_description/urdf/imu.urdf.xacro (robot description, xacro)
@@ -1,7 +1,7 @@
 <?xml version="1.0" ?>
 <robot name="rover" xmlns:xacro="http://www.ros.org/wiki/xacro">
-    <xacro:include filename="$(find rover_description)/urdf/stereo.gazebo.xacro"/>
+    <xacro:include filename="$(find rover_description)/urdf/stereo.imu.xacro"/>
     <xacro:property name="M_PI" value="3.1415926535897931" />
-    <link name="camera_link">
+    <link name="imu_link">
       <collision>
         <origin xyz="0 0 0" rpy="0 0 0"/>

File: src/rover_description/urdf/rover.xacro (robot description, xacro)
@@ -4,4 +4,4 @@
   <xacro:include filename="$(find rover_description)/urdf/rover_description.xacro" />
   <xacro:include filename="$(find rover_description)/urdf/diff_control.xacro" />
-  <xacro:include filename="$(find rover_description)/urdf/rover_camera.xacro" />
+  <xacro:include filename="$(find rover_description)/urdf/rgbd.gazebo.xacro" />
 </robot>

File: src/rover_description/urdf/rover_description.xacro (robot description, xacro)
@@ -1,7 +1,6 @@
 <?xml version="1.0" ?>
 <robot name="rover" xmlns:xacro="http://www.ros.org/wiki/xacro">
-<!-- <xacro:include filename="$(find realsense2_description)/urdf/_d435.urdf.xacro" /> -->
 <material name="silver">
-  <color rgba="0.700 0.700 0.700 1.000"/>
+  <color rgba="1.00 1.00 1.00 1.000"/>
 </material>
 <link name="base_link">
@@ -25,4 +24,7 @@
   </collision>
 </link>
+<gazebo reference="base_link">
+  <material>Gazebo/Orange</material>
+</gazebo>
 <link name="wheel_left_back_1">
   <inertial>
@@ -145,5 +147,5 @@
   </collision>
 </link>
-<joint name="left_back" type="fixed">
+<joint name="left_back" type="continuous">
   <origin xyz="-0.363731 0.088 -0.21" rpy="0 0 0"/>
   <parent link="chassis_left_1"/>
@@ -151,5 +153,5 @@
   <axis xyz="0.0 1.0 -0.0"/>
 </joint>
-<joint name="right_back" type="fixed">
+<joint name="right_back" type="continuous">
   <origin xyz="-0.363731 -0.088 -0.21" rpy="0 0 0"/>
   <parent link="chassis_right_1"/>

File: src/rover_description/urdf/stereo.gazebo.xacro (robot description, xacro)
@@ -1,13 +1,11 @@
 <?xml version="1.0"?>
-<!--
-License: Apache 2.0. See LICENSE file in root directory.
-Copyright(c) 2017 PAL Robotics, S.L. All Rights Reserved
-This is the Gazebo URDF model for the Intel RealSense D435 camera
--->
 <robot xmlns:xacro="http://ros.org/wiki/xacro">
-  <xacro:macro name="gazebo_d435" params="topics_ns" >
+<xacro:macro name="gazebo_d435" params="topics_ns" >
     <!-- Load parameters to model's main link-->
     <xacro:property name="deg_to_rad" value="0.01745329251994329577" />
     <gazebo reference="stereo_camera_left_frame">
+      <gazebo reference="link1">
+        <material>Gazebo/Orange</material>
+      </gazebo>
       <sensor name="stereo_camera_left" type="camera">
         <camera name="stereo_camera_left">

File: src/rover_description/urdf/stereo.urdf.xacro (robot description, xacro)
@@ -1,135 +1,66 @@
-<?xml version="1.0"?>
-<!--
-License: Apache 2.0. See LICENSE file in root directory.
-Copyright(c) 2017 Intel Corporation. All Rights Reserved
-This is the URDF model for the Intel RealSense 430 camera, in it's
-aluminum peripherial evaluation case.
--->
-<robot name="stereo_camera" xmlns:xacro="http://ros.org/wiki/xacro">
-  <!--File includes-->
-  <xacro:include filename="$(find rover_description)/urdf/stereo.gazebo.xacro"/>
-  <xacro:macro name="sensor_d435" params="name:=camera topics_ns:=camera parent *origin publish_pointcloud:=true">
+<?xml version="1.0" ?>
+<robot name="rover" xmlns:xacro="http://www.ros.org/wiki/xacro">
+    <xacro:include filename="$(find rover_description)/urdf/stereo.gazebo.xacro"/>
     <xacro:property name="M_PI" value="3.1415926535897931" />
-    <!-- The following values are approximate, and the camera node
-     publishing TF values with actual calibrated camera extrinsic values -->
-    <xacro:property name="d435_cam_depth_to_left_ir_offset" value="0.0"/>
-    <xacro:property name="d435_cam_depth_to_right_ir_offset" value="-0.050"/>
-    <xacro:property name="d435_cam_depth_to_color_offset" value="0.015"/>
-    <!-- The following values model the aluminum peripherial case for the
-    D435 camera, with the camera joint represented by the actual
-    peripherial camera tripod mount -->
-    <xacro:property name="d435_cam_width" value="0.090"/>
-    <xacro:property name="d435_cam_height" value="0.025"/>
-    <xacro:property name="d435_cam_depth" value="0.02505"/>
-    <xacro:property name="d435_cam_mount_from_center_offset" value="0.0149"/>
-    <!-- The following offset is relative the the physical D435 camera peripherial
-    camera tripod mount -->
-    <xacro:property name="d435_cam_depth_px" value="${d435_cam_mount_from_center_offset}"/>
-    <xacro:property name="d435_cam_depth_py" value="0.0175"/>
-    <xacro:property name="d435_cam_depth_pz" value="${d435_cam_height/2}"/>
-    <material name="${name}_aluminum">
-    <color rgba="0.5 0.5 0.5 1"/>
+    <material name="black">
+      <color rgba="0.00 0.00 0.00 1.000"/>
     </material>
-    <!-- camera body, with origin at bottom screw mount -->
-    <joint name="${name}_joint" type="fixed">
-      <xacro:insert_block name="origin" />
-      <parent link="${parent}"/>
-      <child link="${name}_bottom_screw_frame" />
+    <link name="camera_link"/>
+    <joint name="camera_joint" type="fixed">
+      <axis xyz="0 1 0" />
+      <origin xyz="0.33 0.0 0.4" rpy="0 0 0"/>
+      <parent link="base_link"/>
+      <child link="camera_link"/>
     </joint>
-    <link name="${name}_bottom_screw_frame"/>
-    <joint name="${name}_link_joint" type="fixed">
-      <origin xyz="0 ${d435_cam_depth_py} ${d435_cam_depth_pz}" rpy="0 0 0"/>
-      <parent link="${name}_bottom_screw_frame"/>
-      <child link="${name}_link" />
+    <joint name="left_optical_joint" type="fixed">
+      <origin xyz="0 0 0" rpy="0 0 0" />
+      <parent link="camera_link" />
+      <child link="stereo_camera_left_frame" />
     </joint>
-    <link name="${name}_link">
-      <visual>
-      <origin xyz="${d435_cam_mount_from_center_offset} ${-d435_cam_depth_py} 0" rpy="${M_PI/2} 0 ${M_PI/2}"/>
+    <link name="stereo_camera_left_frame">
+      <collision>
+        <origin xyz="0 0 0" rpy="0 0 0"/>
         <geometry>
-          <!-- <box size="${d435_cam_width} ${d435_cam_height} ${d435_cam_depth}"/> -->
-          <!-- <mesh filename="package://realsense2_description/meshes/d435.dae" /> -->
-          <mesh filename="file://$(find rover_description)/meshes/d435.dae" scale="1 1 1"/>
-        </geometry>
-        <material name="${name}_aluminum"/>
-      </visual>
-      <collision>
-        <origin xyz="0 ${-d435_cam_depth_py} 0" rpy="0 0 0"/>
-        <geometry>
-        <box size="${d435_cam_depth} ${d435_cam_width} ${d435_cam_height}"/>
+          <box size="0.02 0.04 0.02"/>
         </geometry>
       </collision>
+      <visual>
+        <origin xyz="0 0 0" rpy="0 0 0"/>
+        <geometry>
+          <box size="0.02 0.04 0.02"/>
+        </geometry>
+        <material name="black"/>
+      </visual>
       <inertial>
-        <!-- The following are not reliable values, and should not be used for modeling -->
-        <mass value="0.564" />
-        <origin xyz="0 0 0" />
-        <inertia ixx="0.003881243" ixy="0.0" ixz="0.0" iyy="0.000498940" iyz="0.0" izz="0.003879257" />
+        <mass value="1e-5" />
+        <origin xyz="0 0 0" rpy="0 0 0"/>
+        <inertia ixx="1e-6" ixy="0" ixz="0" iyy="1e-6" iyz="0" izz="1e-6" />
       </inertial>
     </link>
-    <!-- camera depth joints and links -->
-    <joint name="${name}_depth_joint" type="fixed">
-      <origin xyz="0 0 0" rpy="0 0 0"/>
-      <parent link="${name}_link"/>
-      <child link="${name}_depth_frame" />
+    <joint name="stereo_camera_right_joint" type="fixed">
+      <origin xyz="-0 -0.05 0" rpy="0 0 0" />
+      <parent link="camera_link" />
+      <child link="stereo_camera_right_frame" />
     </joint>
-    <link name="${name}_depth_frame"/>
-    <joint name="${name}_depth_optical_joint" type="fixed">
-      <origin xyz="0 0 0" rpy="${-M_PI/2} 0 ${-M_PI/2}" />
-      <parent link="${name}_depth_frame" />
-      <child link="${name}_depth_optical_frame" />
-    </joint>
-    <link name="${name}_depth_optical_frame"/>
-    <!-- camera left IR joints and links -->
-    <!-- <joint name="${name}_left_ir_joint" type="fixed">
-      <origin xyz="0 ${d435_cam_depth_to_left_ir_offset} 0" rpy="0 0 0" />
-      <parent link="${name}_depth_frame" />
-      <child link="${name}_left_ir_frame" />
-    </joint>
-    <link name="${name}_left_ir_frame"/>
-    <joint name="${name}_left_ir_optical_joint" type="fixed">
-      <origin xyz="0 0 0" rpy="${-M_PI/2} 0 ${-M_PI/2}" />
-      <parent link="${name}_left_ir_frame" />
-      <child link="${name}_left_ir_optical_frame" />
-    </joint>
-    <link name="${name}_left_ir_optical_frame"/> -->
-    <!-- camera right IR joints and links -->
-    <!-- <joint name="${name}_right_ir_joint" type="fixed">
-      <origin xyz="0 ${d435_cam_depth_to_right_ir_offset} 0" rpy="0 0 0" />
-      <parent link="${name}_depth_frame" />
-      <child link="${name}_right_ir_frame" />
-    </joint>
-    <link name="${name}_right_ir_frame"/>
-    <joint name="${name}_right_ir_optical_joint" type="fixed">
-      <origin xyz="0 0 0" rpy="${-M_PI/2} 0 ${-M_PI/2}" />
-      <parent link="${name}_right_ir_frame" />
-      <child link="${name}_right_ir_optical_frame" />
-    </joint>
-    <link name="${name}_right_ir_optical_frame"/> -->
-    <!-- camera color joints and links -->
-    <joint name="${name}_color_joint" type="fixed">
-      <origin xyz="0 ${d435_cam_depth_to_color_offset} 0" rpy="0 0 0" />
-      <parent link="${name}_depth_frame" />
-      <child link="${name}_color_frame" />
-    </joint>
-    <link name="${name}_color_frame"/>
-    <joint name="${name}_color_optical_joint" type="fixed">
-      <origin xyz="0 0 0" rpy="${-M_PI/2} 0 ${-M_PI/2}" />
-      <parent link="${name}_color_frame" />
-      <child link="${name}_color_optical_frame" />
-    </joint>
-    <link name="${name}_color_optical_frame"/>
-    <joint name="${name}_left_ir_optical_joint" type="fixed">
-      <origin xyz="0 0 0" rpy="${-M_PI/2} 0 ${-M_PI/2}" />
-      <parent link="${parent}" />
-      <child link="${name}_left_ir_optical_frame" />
-    </joint>
-    <link name="${name}_left_ir_optical_frame"/>
-    <joint name="${name}_right_ir_optical_joint" type="fixed">
-      <origin xyz="0 -0.05 0" rpy="${-M_PI/2} 0 ${-M_PI/2}" />
-      <parent link="${parent}" />
-      <child link="${name}_right_ir_optical_frame" />
-    </joint>
-    <link name="${name}_right_ir_optical_frame"/>
-    <!-- Realsense Gazebo Plugin -->
-    <xacro:gazebo_d435 camera_name="${name}" topics_ns="stereo_camera" depth_optical_frame="${name}_depth_optical_frame" color_optical_frame="${name}_color_optical_frame" infrared1_optical_frame="${name}_left_ir_optical_frame" infrared2_optical_frame="${name}_right_ir_optical_frame" publish_pointcloud="${publish_pointcloud}"/>
-  </xacro:macro>
+    <link name="stereo_camera_right_frame">
+      <collision>
+        <origin xyz="0 0 0" rpy="0 0 0"/>
+        <geometry>
+          <box size="0.02 0.04 0.02"/>
+        </geometry>
+      </collision>
+      <visual>
+        <origin xyz="0 0 0" rpy="0 0 0"/>
+        <geometry>
+          <box size="0.02 0.04 0.02"/>
+        </geometry>
+        <material name="black"/>
+      </visual>
+      <inertial>
+        <mass value="1e-5" />
+        <origin xyz="0 0 0" rpy="0 0 0"/>
+        <inertia ixx="1e-6" ixy="0" ixz="0" iyy="1e-6" iyz="0" izz="1e-6" />
+      </inertial>
+    </link>
+    <xacro:gazebo_d435 topics_ns="stereo_camera" />
 </robot>
