Commit message: adjustment for activate ekf

File: src/rover_description/urdf/diff_control.xacro (robot description, xacro)
@@ -6,5 +6,5 @@
       <parameters>$(find rover_description)/config/diff_robot.yaml</parameters>
       <ros>
-        <remapping>/diff_drive_controller/cmd_vel_unstamped:=/cmd_vel</remapping>
+        <remapping>/diff_drive_controller/cmd_vel_unstamped:=/cmd_vel/filtered</remapping>
         <remapping>/diff_drive_controller/odom:=/odom</remapping>
       </ros>

File: src/rover_description/urdf/imu.gazebo.xacro (robot description, xacro)
@@ -1,53 +1,25 @@
 <?xml version="1.0"?>
 <robot xmlns:xacro="http://ros.org/wiki/xacro">
-    <link name="imu_link">
-      <collision>
-        <origin xyz="0 0 0" rpy="0 0 0"/>
-        <geometry>
-          <box size="0.01 0.01 0.01"/>
-        </geometry>
-      </collision>
-      <visual>
-        <origin xyz="0 0 0" rpy="0 0 0"/>
-        <geometry>
-          <box size="0.01 0.01 0.01"/>
-        </geometry>
-        <material name="silver">
-          <color rgba="0.700 0.700 0.700 1.000"/>
-        </material>
-      </visual>
-      <inertial>
-        <mass value="1e-5" />
-        <origin xyz="0 0 0" rpy="0 0 0"/>
-        <inertia ixx="1e-6" ixy="0" ixz="0" iyy="1e-6" iyz="0" izz="1e-6" />
-      </inertial>
-    </link>
-    <joint name="imu_joint" type="fixed">
-      <axis xyz="0 1 0" />
-      <origin xyz="0. 0.0 0.5" rpy="0 0 0"/>
-      <parent link="base_link"/>
-      <child link="imu_link"/>
-    </joint>
-    <gazebo reference="imu_link">
-        <gravity>true</gravity>
-        <sensor name="imu_sensor" type="imu">
-        <always_on>true</always_on>
-        <update_rate>10</update_rate>
-        <visualize>true</visualize>
-        <topic>__default_topic__</topic>
-        <plugin filename="libgazebo_ros_imu_sensor.so" name="imu_plugin">
-            <ros>
-                <remapping>/imu_plugin/out:=/sim/imu</remapping>
-            </ros>
-            <bodyName>imu_link</bodyName>
-            <updateRateHZ>10.0</updateRateHZ>
-            <gaussianNoise>0.0</gaussianNoise>
-            <xyzOffset>0 0 0</xyzOffset>
-            <rpyOffset>0 0 0</rpyOffset>
-            <frameName>imu_link</frameName>
-            <initialOrientationAsReference>false</initialOrientationAsReference>
-        </plugin>
-        <pose>0 0 0 0 0 0</pose>
-        </sensor>
-    </gazebo>
+  <gazebo reference="imu_link">
+      <gravity>true</gravity>
+      <sensor name="imu_sensor" type="imu">
+      <always_on>true</always_on>
+      <update_rate>10</update_rate>
+      <visualize>true</visualize>
+      <topic>__default_topic__</topic>
+      <plugin filename="libgazebo_ros_imu_sensor.so" name="imu_plugin">
+          <ros>
+              <remapping>/imu_plugin/out:=/sim/imu</remapping>
+          </ros>
+          <bodyName>imu_link</bodyName>
+          <updateRateHZ>10.0</updateRateHZ>
+          <gaussianNoise>0.0</gaussianNoise>
+          <xyzOffset>0 0 0</xyzOffset>
+          <rpyOffset>0 0 0</rpyOffset>
+          <frameName>imu_link</frameName>
+          <initialOrientationAsReference>false</initialOrientationAsReference>
+      </plugin>
+      <pose>0 0 0 0 0 0</pose>
+      </sensor>
+  </gazebo>
 </robot>

File: src/rover_description/urdf/rgbd.gazebo.xacro (robot description, xacro)
@@ -1,17 +1,4 @@
 <?xml version="1.0"?>
 <robot xmlns:xacro="http://ros.org/wiki/xacro">
-    <!-- Load parameters to model's main link-->
-    <link name="camera_link"/>
-    <link name="depth_link"/>
-    <joint name="base_to_camera" type="fixed">
-      <origin xyz="0.35 0.0 0.4" rpy="0 0 0"/>
-      <parent link="base_link"/>
-      <child link="camera_link"/>
-    </joint>
-    <joint name="camera_to_depth" type="fixed">
-      <origin xyz="0.0 0.0 0.0" rpy="-1.5707 0 -1.5707"/>
-      <parent link="camera_link"/>
-      <child link="depth_link"/>
-    </joint>
     <gazebo reference="camera_link">
       <gazebo reference="link1">
@@ -60,5 +47,5 @@
               <width>1280</width>
               <height>720</height>
-              <format>R8G8B8</format>
+              <format>RGB_INT8</format>
             </image>
             <horizontal_fov>1.57</horizontal_fov>
@@ -76,5 +63,5 @@
             <hack_baseline>0.07</hack_baseline>
             <min_depth>0.4</min_depth>
-            <max_depth>20.0</max_depth>
+            <max_depth>200.0</max_depth>
           </plugin>
         </sensor>

File: src/rover_description/urdf/rover.xacro (robot description, xacro)
@@ -2,5 +2,7 @@
 <robot name="rover" xmlns:xacro="http://www.ros.org/wiki/xacro">
   <xacro:include filename="$(find rover_description)/urdf/rover.trans" />
+  <!-- <xacro:include filename="$(find rover_description)/urdf/unit2.trans" /> -->
   <xacro:include filename="$(find rover_description)/urdf/rover_description.xacro" />
+  <!-- <xacro:include filename="$(find rover_description)/urdf/unit2_description.xacro" /> -->
   <xacro:include filename="$(find rover_description)/urdf/diff_control.xacro" />
   <xacro:include filename="$(find rover_description)/urdf/rgbd.gazebo.xacro" />

File: src/rover_description/urdf/rover_description.xacro (robot description, xacro)
@@ -183,3 +183,45 @@
   <axis xyz="0.0 -1.0 0.0"/>
 </joint>
+<!-- camera -->
+<link name="camera_link"/>
+<link name="depth_link"/>
+<joint name="base_to_camera" type="fixed">
+  <origin xyz="0.35 0.0 0.4" rpy="0 0 0"/>
+  <parent link="base_link"/>
+  <child link="camera_link"/>
+</joint>
+<joint name="camera_to_depth" type="fixed">
+  <origin xyz="0.0 0.0 0.0" rpy="-1.5707 0 -1.5707"/>
+  <parent link="camera_link"/>
+  <child link="depth_link"/>
+</joint>
+<!-- imu -->
+<link name="imu_link">
+  <collision>
+    <origin xyz="0 0 0" rpy="0 0 0"/>
+    <geometry>
+      <box size="0.01 0.01 0.01"/>
+    </geometry>
+  </collision>
+  <visual>
+    <origin xyz="0 0 0" rpy="0 0 0"/>
+    <geometry>
+      <box size="0.01 0.01 0.01"/>
+    </geometry>
+    <material name="silver">
+      <color rgba="0.700 0.700 0.700 1.000"/>
+    </material>
+  </visual>
+  <inertial>
+    <mass value="1e-5" />
+    <origin xyz="0 0 0" rpy="0 0 0"/>
+    <inertia ixx="1e-6" ixy="0" ixz="0" iyy="1e-6" iyz="0" izz="1e-6" />
+  </inertial>
+</link>
+<joint name="imu_joint" type="fixed">
+  <axis xyz="0 1 0" />
+  <origin xyz="0. 0.0 0.5" rpy="0 0 0"/>
+  <parent link="base_link"/>
+  <child link="imu_link"/>
+</joint>
 </robot>
