Commit message: inactivate gazebo sensor joints

File: src/rover_description/urdf/unit2_description.xacro (robot description, xacro)
@@ -134,5 +134,5 @@
   </collision>
 </link>
-<joint name="left_back" type="continuous">
+<joint name="left_back" type="fixed">
   <origin xyz="-0.200297 0.0 -0.166452" rpy="0 0 0"/>
   <parent link="unit2_left_chasis_1"/>
@@ -140,5 +140,5 @@
   <axis xyz="-0.0 1.0 0.0"/>
 </joint>
-<joint name="left_front" type="continuous">
+<joint name="left_front" type="fixed">
   <origin xyz="0.188382 0.013 -0.179825" rpy="0 0 0"/>
   <parent link="unit2_left_chasis_1"/>
@@ -160,5 +160,5 @@
   <limit upper="0.523599" lower="-0.523599" effort="100" velocity="100"/>
 </joint>
-<joint name="right_front" type="continuous">
+<joint name="right_front" type="fixed">
   <origin xyz="0.194454 -0.0035 -0.173241" rpy="0 0 0"/>
   <parent link="unit2_right_chasis_1"/>
@@ -166,5 +166,5 @@
   <axis xyz="0.0 1.0 -0.0"/>
 </joint>
-<joint name="right_back" type="continuous">
+<joint name="right_back" type="fixed">
   <origin xyz="-0.194454 -0.0165 -0.173241" rpy="0 0 0"/>
   <parent link="unit2_right_chasis_1"/>
@@ -172,6 +172,6 @@
   <axis xyz="0.0 1.0 -0.0"/>
 </joint>
-<!-- camera -->
-<link name="camera_link"/>
+<!-- gazebo_camera -->
+<!-- <link name="camera_link"/>
 <link name="depth_link"/>
 <joint name="base_to_camera" type="fixed">
@@ -184,7 +184,7 @@
   <parent link="camera_link"/>
   <child link="depth_link"/>
-</joint>
+</joint> -->
 <!-- imu -->
-<link name="imu_link">
+<!-- <link name="imu_link">
   <collision>
     <origin xyz="0 0 0" rpy="0 0 0"/>
@@ -213,4 +213,4 @@
   <parent link="base_link"/>
   <child link="imu_link"/>
-</joint>
+</joint> -->
 </robot>
